Commit message: Moved from DH to URDF models, added PSM
Minor fixes to URDF files, improved test script, and moved friction into utils

File: models/mtm/mtm.urdf.xacro (robot description, xacro)
@@ -2,5 +2,5 @@
 <robot name="mtm" xmlns:xacro="http://www.ros.org/wiki/xacro">
   <!-- Colors -->
-  <xacro:include filename="$(find dvrk_description)/mtm/common.urdf.xacro"/>
+  <xacro:include filename="common.urdf.xacro"/>
   <!-- Macro for the da Vinci Master Console -->
   <xacro:macro name="master_console" params="prefix parent_link xyz rpy">
@@ -112,5 +112,5 @@
       </inertial>
     </link>
-     <!--link name="${prefix}front_parallel_link">
+     <link name="${prefix}front_parallel_link">
        <visual>
          <geometry>
@@ -127,5 +127,5 @@
          <inertia ixx="8.0" ixy="0.0" ixz="0.0" iyy="8.0" iyz="0.0" izz="8.0"/>
        </inertial>
-     </link-->
+     </link>
     <joint name="${prefix}shoulder_pitch_joint" type="revolute">
       <parent link="${prefix}outer_yaw_link"/>
@@ -149,5 +149,5 @@
       <mimic joint="${prefix}elbow_pitch_joint" multiplier="1"/>
     </joint>
-    <!--joint name="${prefix}elbow_pitch_parallel_joint" type="revolute">
+    <joint name="${prefix}elbow_pitch_parallel_joint" type="revolute">
        <parent link="${prefix}top_parallel_link"/>
        <child link="${prefix}front_parallel_link"/>
@@ -157,5 +157,5 @@
        <joint_properties damping="1.0" friction="0.0"/>
        <mimic joint="${prefix}elbow_pitch_joint" multiplier="-1"/>
-     </joint-->
+     </joint>
     <joint name="${prefix}elbow_pitch_joint" type="revolute">
       <parent link="${prefix}back_parallel_link"/>

File: models/mtm/mtm_launch.urdf.xacro (robot description, xacro)
@@ -2,5 +2,5 @@
 <robot name="master" xmlns:xacro="http://www.ros.org/wiki/xacro">
   <!-- Macros -->
-  <xacro:include filename="$(find dvrk_description)/mtm/mtm.urdf.xacro"/>
+  <xacro:include filename="mtm.urdf.xacro"/>
   <link name="world"/>
   <xacro:mtm

File: models/psm/psm_launch.urdf.xacro (robot description, xacro)
@@ -1,5 +1,5 @@
 <?xml version="1.0" ?>
 <robot name="master" xmlns:xacro="http://www.ros.org/wiki/xacro">
-<xacro:include filename="$(find dvrk_description)/psm/psm.urdf.xacro"/>
+<xacro:include filename="psm.urdf.xacro"/>
 <link name="world"/>
 <xacro:psm parent_link="world" prefix="psm_" xyz="0 0 0.1524" rpy="0 0 0"/>
